File: Platine/HB-OU-RGB-STACKFIRE (Mega2560)V2/HB-OU-RGB-STACKFIRE.kicad_pcb (KiCad board)
At the start: 2 copper layers, 193 x 193 mm, 34 parts, among them J1 230V, J11 Stackfire-Ring, J12 230V (OUT 2), J2 230V (OUT 1), J3 LLV, J4 LLV, J5 5V - WS28XX, J6 5V - WS28XX, J8 5V - WS28XX, J9 5V - WS28XX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

Commit message: V3
Parts:
- removed J11: Stackfire-Ring, Homebrew:Stackfire-Ring
- removed J12: 230V (OUT 2), TerminalBlock_WAGO:TerminalBlock_WAGO_236-103_1x03_P5.00mm_45Degree
- added J7: 5V - WS28XX, digikey-footprints:PinHeader_1x2_P3.96mm_Drill1.6mm, F.Cu at (125.9, 159.6)
- added U1: CC1101, Homebrew:CC1101, F.Cu at (251.6, 141.0)
- C1: value 100nF -> 10uF; footprint Capacitor_THT:C_Disc_D5.0mm_W2.5mm_P2.50mm -> Capacitor_THT:CP_Radial_D5.0mm_P2.50mm
- C2: value 10uF -> 100nF; footprint Capacitor_THT:CP_Radial_D5.0mm_P2.50mm -> Capacitor_THT:C_Disc_D5.0mm_W2.5mm_P2.50mm
- Cp1: value Version 2.0.1 - 01/2020 -> Version 2.0.1 - 02/2020
- J1: value 230V -> 230V (OUT 1)
- J2: value 230V (OUT 1) -> 230V
- J3: value LLV -> 230V (OUT 2); footprint Connector_PinHeader_2.54mm:PinHeader_1x06_P2.54mm_Vertical -> TerminalBlock_WAGO:TerminalBlock_WAGO_236-103_1x03_P5.00mm_45Degree; moved to B.Cu
- J4: value LLV -> VCC; footprint Connector_PinHeader_2.54mm:PinHeader_1x06_P2.54mm_Vertical -> Connector_PinHeader_2.54mm:PinHeader_2x02_P2.54mm_Vertical
- J5, J6, J8: moved to F.Cu
- J9: value 5V - WS28XX -> Stackfire-Ring; footprint digikey-footprints:PinHeader_1x2_P3.96mm_Drill1.6mm -> Homebrew:Stackfire-Ring; moved to F.Cu
- U2: value CC1101 -> 8-Kanal_LevelShifter; footprint Homebrew:CC1101 -> Homebrew:Adafruit 8-Kanal Level Shifter
- moved J3 167.5 mm to (96.5, 185.2), turned to 180 degrees
- moved C1 114.9 mm to (260.4, 137.2), turned to 0 degrees
- moved J4 112.7 mm to (136.9, 122.3), turned to 0 degrees
- moved C2 110.5 mm to (151.0, 101.6), turned to 90 degrees
- moved J6 96.1 mm to (220.2, 177.5), turned to 255 degrees
- moved J9 48.2 mm to (173.9, 164.4), turned to 0 degrees
- moved SW1 34.2 mm to (158.1, 112.6), turned to 90 degrees
- moved D1 25.1 mm to (158.1, 101.7), turned to 90 degrees
- moved R1 20.3 mm to (163.7, 99.2)
- moved MH3 19.6 mm to (221.4, 230.1)
- moved MH2 18.6 mm to (236.2, 180.7)
- moved MH1 9.09 mm to (242.1, 161.5)
- moved U2 4.50 mm to (245.0, 130.8), turned to 90 degrees
- moved J5 3.98 mm to (151.8, 121.5), turned to 26 degrees
- moved J8 3.91 mm to (202.9, 202.8), turned to 215 degrees
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Connections:
- B1 pad 13: /WS28XX_6 -> Net-(B1-Pad13)
- B1 pad 15: /WS28XX_7 -> /WS28XX_6
- B1 pad 17: /WS28XX_8 -> /WS28XX_7
- B1 pad 19: /WS28XX_9 -> /WS28XX_8
- B1 pad 2: /D2 -> /HV5(D2)
- B1 pad 20: Net-(B1-Pad20) -> /WS28XX_9
- C1 pad 1: +VDC -> +3V3
- C2 pad 1: +3V3 -> +VDC
- J1 pad 1: Net-(F1-Pad1) -> Net-(F1-Pad2)
- J2 pad 1: Net-(F1-Pad1) -> Net-(F1-Pad2)
- J3 pad 1: /HV4(SS) -> Net-(F1-Pad1)
- J3 pad 2: /HV3(SCK) -> Net-(J1-Pad2)
- J3 pad 3: GND -> Net-(J1-Pad3)
- J4 pad 1: /LV4(SS) -> +VDC
- J4 pad 2: /LV3(SCK) -> GND
- J4 pad 3: GND -> /VCC_WS28XX_1_1
- J4 pad 4: +3V3 -> GND
- J8 pad 2: /VCC_WS28XX_2_1 -> /VCC_WS28XX_2_2
- J9 pad 2: /VCC_WS28XX_2_2 -> /WS28XX_1
- PS1 pad 1: Net-(F1-Pad2) -> Net-(J1-Pad2)
- PS1 pad 2: Net-(J1-Pad2) -> Net-(F1-Pad2)
- SW1 pad 1: GND -> Net-(B1-Pad13)
- SW1 pad 2: Net-(B1-Pad8) -> GND
- U2 pad 2: GND -> /LV4(SS)
- U2 pad 3: /LV2(MOSI) -> /LV5(D2)
- U2 pad 4: /LV3(SCK) -> Net-(U2-Pad4)
- U2 pad 7: /D2 -> /LV3(SCK)
- U2 pad 8: /LV4(SS) -> Net-(U2-Pad8)
Routing:
- net /VCC_WS28XX_2_1: track 78.3 -> 191.9 mm
- net /VCC_WS28XX_1_2: track 78.6 -> 186.8 mm
- net /VCC_WS28XX_1_1: track 76.4 -> 143.4 mm
- net /D2: track 61.5 -> 0.00 mm
- net Net-(B1-Pad8): track 59.9 -> 0.00 mm
- net /HV5(D2): track 0.00 -> 57.8 mm
- net Net-(B1-Pad13): track 0.00 -> 49.8 mm
- net /VCC_WS28XX_2_2: track 85.1 -> 127.4 mm
- net +5V: track 89.5 -> 65.6 mm
- net Net-(F1-Pad1): track 83.9 -> 62.2 mm
- net Net-(B1-Pad4): track 45.0 -> 29.2 mm
- net /LV4(SS): track 21.8 -> 6.31 mm
- net /WS28XX_13: track 74.4 -> 88.4 mm
- net /WS28XX_9: track 93.0 -> 106.9 mm
- net +VDC: track 37.8 -> 51.6 mm
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Other:
- board text added: "ACHTUNG !!! Jumper nur bei fehlendem Netzteil stecken"
- board text added: "GND"
- board text removed: "NT 1/3"
- board text removed: "NT 2/3"
