File: Platine/HB-OU-RGB-STACKFIRE (Mega2560)V2/HB-OU-RGB-STACKFIRE.sch (KiCad schematic (older format))
At the start: 20 parts, among them J1 230V, J11 Stackfire-Ring, J12 230V (OUT 2), J2 230V (OUT 1), J3 LLV, J4 LLV, J5 5V - WS28XX, J6 5V - WS28XX, J8 5V - WS28XX, J9 5V - WS28XX, SW1 CONFIG, U2 CC1101

Commit message: V3
Parts:
- removed J3, J4: LLV, Connector_PinHeader_2.54mm:PinHeader_1x06_P2.54mm_Vertical, symbol Connector_Generic:Conn_01x06
- added J4: VCC, Connector_PinHeader_2.54mm:PinHeader_2x02_P2.54mm_Vertical, symbol Connector_Generic:Conn_02x02_Counter_Clockwise
- added U2: 8-Kanal_LevelShifter, Homebrew:Adafruit 8-Kanal Level Shifter, symbol Homebrew:8-Kanal_LevelShifter
- renumbered C2 to C1, C1 to C2, J2 to J1, J1 to J2, J12 to J3, J8 to J7, J9 to J8, J11 to J9, U2 to U1
Connections:
- net +3V3: now also U2.1 (VA), U2.10 (OE)
- net +5V: now also U2.11 (VB)
- net +VDC: now also J4.1 (Pin_1)
- net GND: now also SW1.2, J4.2 (Pin_2), J4.4 (Pin_4), U2.20 (GND); no longer SW1.1
- net HV1(MISO): now also U2.15 (B4)
- net HV2(MOSI): now also U2.19 (B8)
- net HV3(SCK): now also U2.17 (B6)
- net HV4(SS): now also U2.12 (B1)
- net LV1(MISO): now also U2.5 (A4)
- net LV2(MOSI): now also U2.9 (A8)
- net LV3(SCK): now also U2.7 (A6)
- net LV4(SS): now also U2.2 (A1)
- net VCC_WS28XX_1_1: now also J9.74 (VCC_WS28XX), J9.78 (VCC_WS28XX), J4.3 (Pin_3); no longer J9.64 (VCC_WS28XX), J9.68 (VCC_WS28XX)
- net VCC_WS28XX_1_2: now also J9.82 (VCC_WS28XX), J9.86 (VCC_WS28XX), J9.90 (VCC_WS28XX), J9.94 (VCC_WS28XX), J9.98 (VCC_WS28XX); no longer J9.72 (VCC_WS28XX), J9.74 (VCC_WS28XX), J9.76 (VCC_WS28XX), J9.78 (VCC_WS28XX), J9.80 (VCC_WS28XX)
- net VCC_WS28XX_2_1: now also J9.64 (VCC_WS28XX), J9.68 (VCC_WS28XX), J9.72 (VCC_WS28XX), J9.76 (VCC_WS28XX), J9.80 (VCC_WS28XX); no longer J9.82 (VCC_WS28XX), J9.84 (VCC_WS28XX), J9.86 (VCC_WS28XX), J9.88 (VCC_WS28XX), J9.90 (VCC_WS28XX)
- net VCC_WS28XX_2_2: now also J9.84 (VCC_WS28XX), J9.88 (VCC_WS28XX); no longer J9.94 (VCC_WS28XX), J9.98 (VCC_WS28XX)
- net WS28XX_6: now also B1.15 (15(RX3)); no longer B1.13
- net WS28XX_7: now also B1.17 (17(RX2)); no longer B1.15 (15(RX3))
- net WS28XX_8: now also B1.19 (19(RX1)); no longer B1.17 (17(RX2))
- net WS28XX_9: now also B1.20 (20(SDA)); no longer B1.19 (19(RX1))
- net at B1.8: no longer SW1.2
- net at F1.1, J3.1 (Pin_1): no longer J1.1 (Pin_1), J2.1 (Pin_1)
- net at F1.2, RV1.1: now also J1.1 (Pin_1), J2.1 (Pin_1), PS1.2 (AC); no longer PS1.1 (AC)
- net at J1.2 (Pin_2), J2.2 (Pin_2), J3.2 (Pin_2)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: now also PS1.1 (AC); no longer PS1.2 (AC)
- net D2 renamed HV5(D2)
- net HV5(D2): now also U2.13 (B2); no longer U1.7 (GDO0)
- new net: B1.13, SW1.1
- new net LV5(D2): U1.7 (GDO0), U2.3 (A2)
- no-connect marks 48 -> 55
Other:
- note removed: "SparkFun Logical Level Converter\n"
- moved on the sheet: J1, J2, SW1
