File: Platine/HB-OU-RGB-STACKFIRE (Mega2560 + external Button)-V3/HB-OU-RGB-STACKFIRE-V3.sch (KiCad schematic (older format))
At the start: 20 parts, among them J1 230V (OUT 1), J2 230V, J3 230V (OUT 2), J4 VCC, J5 5V - WS28XX, J6 5V - WS28XX, J7 5V - WS28XX, J8 5V - WS28XX, J9 Stackfire-Ring, SW1 CONFIG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

Commit message: Rev 3.0.1 wit external Button (Test)
Parts:
- added SW2: External Button, Connector_PinHeader_2.54mm:PinHeader_1x02_P2.54mm_Vertical, symbol Switch:SW_DIP_x01
Connections:
- net GND: now also SW2.2
- net at F1.2, J1.1 (Pin_1), J2.1 (Pin_1)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: now also PS1.2 (AC); no longer PS1.1 (AC)
- net at J1.2 (Pin_2), J2.2 (Pin_2), J3.2 (Pin_2)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: now also PS1.1 (AC); no longer PS1.2 (AC)
- net at B1.33: now also SW2.1
- no-connect marks 55 -> 54
Changed lines of the file:
@@
 EESchema Schematic File Version 4
-LIBS:HB-OU-RGB-STACKFIRE-cache
+LIBS:HB-OU-RGB-STACKFIRE-V3-cache
 EELAYER 26 0
 EELAYER END
@@
 Sheet 1 1
 Title "HB-OU-RGB-STACKFIRE"
-Date "2020-01-20"
-Rev ""
+Date "2020-02-24"
+Rev "3.0.1"
 Comp ""
-Comment1 ""
-Comment2 ""
-Comment3 ""
-Comment4 ""
+Comment1 "©S. Sternitzke"
+Comment2 "with external Button"
+Comment3 "Bauart: Röhre Plexiglas XT satiniert (Ø200/194mm)"
+Comment4 "Feuersimulation mit WS2812B"
 $EndDescr
 $Comp
@@
 	2045 6880 2220 6880
 Wire Wire Line
-	2320 7280 2320 7180
-Wire Wire Line
-	2045 7180 2320 7180
+	2045 7180 2140 7180
 $Comp
 L Homebrew:TSP-05 PS1
@@
 Wire Wire Line
 	4045 2755 3460 2755
-NoConn ~ 3460 3055
 NoConn ~ 3460 3255
 NoConn ~ 3460 3455
@@
 	1310 7705 1160 7705
 Wire Wire Line
-	1260 7285 2320 7285
-Wire Wire Line
-	2320 7285 2320 7280
+	1310 7385 2220 7385
+Wire Wire Line
+	2220 7385 2220 7280
+Connection ~ 1310 7385
+Wire Wire Line
+	2320 7280 2220 7280
+Connection ~ 2220 7280
+Wire Wire Line
+	2220 7280 2220 6880
+Wire Wire Line
+	1260 7285 2140 7285
+Wire Wire Line
+	2140 7285 2140 7180
 Connection ~ 1260 7285
-Connection ~ 2320 7280
-Wire Wire Line
-	1310 7385 2220 7385
-Wire Wire Line
-	2220 7385 2220 6880
-Connection ~ 1310 7385
-Connection ~ 2220 6880
-Wire Wire Line
-	2220 6880 2320 6880
+Connection ~ 2140 7180
+Wire Wire Line
+	2320 7180 2320 6880
+Wire Wire Line
+	2140 7180 2320 7180
+$Comp
+L Switch:SW_DIP_x01 SW2
+U 1 1 5E553CE5
+P 3885 3055
+F 0 "SW2" H 4130 3135 50  0000 C CNN
+F 1 "External Button" H 3885 2910 50  0000 C CNN
+F 2 "Connector_PinHeader_2.54mm:PinHeader_1x02_P2.54mm_Vertical" H 3885 3055 50  0001 C CNN
+F 3 "" H 3885 3055 50  0001 C CNN
+	1    3885 3055
+	1    0    0    -1
+$EndComp
+Wire Wire Line
+	3460 3055 3585 3055
+$Comp
+L power:GND #PWR?
+U 1 1 5E5822DA
+P 4300 3075
+F 0 "#PWR?" H 4300 2825 50  0001 C CNN
+F 1 "GND" H 4305 2902 50  0000 C CNN
+F 2 "" H 4300 3075 50  0001 C CNN
+F 3 "" H 4300 3075 50  0001 C CNN
+	1    4300 3075
+	1    0    0    -1
+$EndComp
+Wire Wire Line
+	4185 3055 4300 3055
+Wire Wire Line
+	4300 3055 4300 3075
 $EndSCHEMATC
